File: MCP9808/MCP9808.sch (KiCad schematic (older format))
At the start: 14 parts, among them J1 Conn_01x05, U1 MCP9808

Commit message: Part Numbers Added
Parts:
- C1: Part (none) -> C29936
- R1, R6: Part (none) -> C99782
- R2: value 4K7 -> 10K; Part (none) -> C99198
- R3, R4, R5: Part (none) -> C99198
- U1: Part (none) -> C94847
Changed lines of the file:
@@
 F 2 "Resistor_SMD:R_0603_1608Metric" V 1540 1540 50  0001 C CNN
 F 3 "~" H 1500 1550 50  0001 C CNN
+F 4 "C99782" V 1500 1550 50  0001 C CNN "Part"
 	1    1500 1550
 	-1   0    0    -1
@@
 F 2 "Resistor_SMD:R_0603_1608Metric" V 1240 1540 50  0001 C CNN
 F 3 "~" H 1200 1550 50  0001 C CNN
+F 4 "C99782" V 1200 1550 50  0001 C CNN "Part"
 	1    1200 1550
 	-1   0    0    -1
@@
 P 2500 1700
 F 0 "R2" V 2703 1700 50  0000 C CNN
-F 1 "4K7" V 2613 1700 50  0000 C CNN
+F 1 "10K" V 2613 1700 50  0000 C CNN
 F 2 "Resistor_SMD:R_0603_1608Metric" V 2540 1690 50  0001 C CNN
 F 3 "~" H 2500 1700 50  0001 C CNN
+F 4 "C99198" V 2500 1700 50  0001 C CNN "Part"
 	1    2500 1700
 	-1   0    0    -1
@@
 F 2 "Resistor_SMD:R_0603_1608Metric" V 3490 2090 50  0001 C CNN
 F 3 "~" H 3450 2100 50  0001 C CNN
+F 4 "C99198" H 3450 2100 50  0001 C CNN "Part"
 	1    3450 2100
 	-1   0    0    -1
@@
 F 2 "Resistor_SMD:R_0603_1608Metric" V 3690 2090 50  0001 C CNN
 F 3 "~" H 3650 2100 50  0001 C CNN
+F 4 "C99198" H 3650 2100 50  0001 C CNN "Part"
 	1    3650 2100
 	-1   0    0    -1
@@
 F 2 "Resistor_SMD:R_0603_1608Metric" V 3890 2090 50  0001 C CNN
 F 3 "~" H 3850 2100 50  0001 C CNN
+F 4 "C99198" H 3850 2100 50  0001 C CNN "Part"
 	1    3850 2100
 	-1   0    0    -1
@@
 F 2 "Package_SO:MSOP-8_3x3mm_P0.65mm" H 1000 1600 50  0001 C CNN
 F 3 "http://ww1.microchip.com/downloads/en/DeviceDoc/22203b.pdf" H 1750 2550 50  0001 C CNN
+F 4 "C94847" H 2000 2100 50  0001 C CNN "Part"
 	1    2000 2100
 	1    0    0    -1
@@
 F 2 "Capacitor_SMD:C_0603_1608Metric" H 2938 1550 50  0001 C CNN
 F 3 "~" H 2900 1700 50  0001 C CNN
+F 4 "C29936" H 2900 1700 50  0001 C CNN "Part"
 	1    2900 1700
 	1    0    0    -1
