File: BME280/BME280.sch (KiCad schematic (older format))
At the start: 19 parts, among them J1 Conn_01x07, Q1 BSS138DW, Q2 BSS138DW, U1 AP2127K-3.3, U2 BME280

Commit message: Part Numbers Added
Parts:
- C1: Part (none) -> C29936
- C2: part (none) -> C29936
- D1: Part (none) -> C118330
- Q2: Part (none) -> C193381
- R1, R2, R3, R4, R5, R7, R8, R9: Part (none) -> C99198
- R6: Part (none) -> C25585
- U1: Part (none) -> C156285
- U2: Part  (none) -> C92489
Changed lines of the file:
@@
 F 2 "Capacitor_SMD:C_0603_1608Metric" H 4988 1150 50  0001 C CNN
 F 3 "~" H 4950 1300 50  0001 C CNN
+F 4 "C29936" H 4950 1300 50  0001 C CNN "Part"
 	1    4950 1300
 	1    0    0    -1
@@
 F 2 "Capacitor_SMD:C_0603_1608Metric" H 6238 1150 50  0001 C CNN
 F 3 "~" H 6200 1300 50  0001 C CNN
+F 4 "C29936" H 6200 1300 50  0001 C CNN "part"
 	1    6200 1300
 	1    0    0    -1
@@
 F 2 "Resistor_SMD:R_0603_1608Metric" V 6640 1140 50  0001 C CNN
 F 3 "~" H 6600 1150 50  0001 C CNN
+F 4 "C25585" V 6600 1150 50  0001 C CNN "Part"
 	1    6600 1150
 	1    0    0    -1
@@
 F 2 "LED_SMD:LED_0603_1608Metric" H 6600 1550 50  0001 C CNN
 F 3 "~" H 6600 1550 50  0001 C CNN
+F 4 "C118330" H 6600 1550 50  0001 C CNN "Part"
 	1    6600 1550
 	0    -1   -1   0
@@
 F 2 "Package_TO_SOT_SMD:SOT-363_SC-70-6" H 3200 1950 50  0001 C CNN
 F 3 "~" H 3200 1950 50  0001 C CNN
+F 4 "C193381" H 3000 1950 50  0001 C CNN "Part"
 	1    3000 1950
 	1    0    0    -1
@@
 F 2 "Package_TO_SOT_SMD:SOT-363_SC-70-6" H 4000 1950 50  0001 C CNN
 F 3 "~" H 4000 1950 50  0001 C CNN
+F 4 "C193381" H 3800 1950 50  0001 C CNN "Part"
 	2    3800 1950
 	1    0    0    -1
@@
 F 2 "Package_TO_SOT_SMD:SOT-23-5" H 5600 1325 50  0001 C CNN
 F 3 "https://www.diodes.com/assets/Datasheets/AP2127.pdf" H 5600 1100 50  0001 C CNN
+F 4 "C156285" H 5600 1000 50  0001 C CNN "Part"
 	1    5600 1000
 	1    0    0    -1
@@
 F 2 "Resistor_SMD:R_0603_1608Metric" V 3140 1240 50  0001 C CNN
 F 3 "~" H 3100 1250 50  0001 C CNN
+F 4 "C99198" H 3100 1250 50  0001 C CNN "Part"
 	1    3100 1250
 	1    0    0    -1
@@
 F 2 "Resistor_SMD:R_0603_1608Metric" V 3940 1240 50  0001 C CNN
 F 3 "~" H 3900 1250 50  0001 C CNN
+F 4 "C99198" H 3900 1250 50  0001 C CNN "Part"
 	1    3900 1250
 	1    0    0    -1
@@
 F 2 "Resistor_SMD:R_0603_1608Metric" V 2890 2340 50  0001 C CNN
 F 3 "~" H 2850 2350 50  0001 C CNN
+F 4 "C99198" V 2850 2350 50  0001 C CNN "Part"
 	1    2850 2350
 	0    1    1    0
@@
 F 2 "Resistor_SMD:R_0603_1608Metric" V 3640 2340 50  0001 C CNN
 F 3 "~" H 3600 2350 50  0001 C CNN
+F 4 "C99198" V 3600 2350 50  0001 C CNN "Part"
 	1    3600 2350
 	0    1    1    0
@@
 F 2 "Resistor_SMD:R_0603_1608Metric" V 1590 1240 50  0001 C CNN
 F 3 "~" H 1550 1250 50  0001 C CNN
+F 4 "C99198" H 1550 1250 50  0001 C CNN "Part"
 	1    1550 1250
 	1    0    0    -1
@@
 F 2 "Resistor_SMD:R_0603_1608Metric" V 2390 1240 50  0001 C CNN
 F 3 "~" H 2350 1250 50  0001 C CNN
+F 4 "C99198" H 2350 1250 50  0001 C CNN "Part"
 	1    2350 1250
 	1    0    0    -1
@@
 F 2 "Resistor_SMD:R_0603_1608Metric" V 1340 2340 50  0001 C CNN
 F 3 "~" H 1300 2350 50  0001 C CNN
+F 4 "C99198" V 1300 2350 50  0001 C CNN "Part"
 	1    1300 2350
 	0    1    1    0
@@
 F 2 "Resistor_SMD:R_0603_1608Metric" V 2090 2340 50  0001 C CNN
 F 3 "~" H 2050 2350 50  0001 C CNN
+F 4 "C99198" V 2050 2350 50  0001 C CNN "Part"
 	1    2050 2350
 	0    1    1    0
@@
 F 2 "Package_LGA:Bosch_LGA-8_2.5x2.5mm_P0.65mm_ClockwisePinNumbering" H 4950 2850 50  0001 C CNN
 F 3 "https://ae-bst.resource.bosch.com/media/_tech/media/datasheets/BST-BME280_DS001-11.pdf" H 4950 2850 50  0001 C CNN
+F 4 "C92489" H 4950 3050 50  0001 C CNN "Part "
 	1    4950 3050
 	1    0    0    -1

Commit message: BME280 Part number edits
Parts:
- C2: Part (none) -> C29936; part C29936 -> (none)
- Q1: Part (none) -> C193381
- Q2: Part C193381 -> (none)
- U2: Part  C92489 -> (none)
Changed lines of the file:
@@
 F 2 "Capacitor_SMD:C_0603_1608Metric" H 6238 1150 50  0001 C CNN
 F 3 "~" H 6200 1300 50  0001 C CNN
-F 4 "C29936" H 6200 1300 50  0001 C CNN "part"
+F 4 "C29936" H 6200 1300 50  0001 C CNN "Part"
 	1    6200 1300
 	1    0    0    -1
@@
 F 2 "Package_TO_SOT_SMD:SOT-363_SC-70-6" H 4000 1950 50  0001 C CNN
 F 3 "~" H 4000 1950 50  0001 C CNN
-F 4 "C193381" H 3800 1950 50  0001 C CNN "Part"
 	2    3800 1950
 	1    0    0    -1
@@
 F 2 "Package_TO_SOT_SMD:SOT-363_SC-70-6" H 1650 1950 50  0001 C CNN
 F 3 "~" H 1650 1950 50  0001 C CNN
+F 4 "C193381" H 1450 1950 50  0001 C CNN "Part"
 	1    1450 1950
 	1    0    0    -1
@@
 	1    0    0    -1
 $EndComp
-$Comp
-L Sensor:BME280 U2
-U 1 1 5DEB7D0F
-P 4950 3050
-F 0 "U2" H 4520 3095 50  0000 R CNN
-F 1 "BME280" H 4520 3005 50  0000 R CNN
-F 2 "Package_LGA:Bosch_LGA-8_2.5x2.5mm_P0.65mm_ClockwisePinNumbering" H 4950 2850 50  0001 C CNN
-F 3 "https://ae-bst.resource.bosch.com/media/_tech/media/datasheets/BST-BME280_DS001-11.pdf" H 4950 2850 50  0001 C CNN
-F 4 "C92489" H 4950 3050 50  0001 C CNN "Part "
-	1    4950 3050
-	1    0    0    -1
-$EndComp
 Connection ~ 4950 2450
 Wire Wire Line
@@
 	1    0    0    -1
 $EndComp
+$Comp
+L Sensor:BME280 U2
+U 1 1 5DF129EC
+P 4950 3050
+F 0 "U2" H 4520 3095 50  0000 R CNN
+F 1 "BME280" H 4520 3005 50  0000 R CNN
+F 2 "Package_LGA:Bosch_LGA-8_2.5x2.5mm_P0.65mm_ClockwisePinNumbering" H 4950 2850 50  0001 C CNN
+F 3 "https://ae-bst.resource.bosch.com/media/_tech/media/datasheets/BST-BME280_DS001-11.pdf" H 4950 2850 50  0001 C CNN
+	1    4950 3050
+	1    0    0    -1
+$EndComp
