File: ADXL345/ADXL345.sch (KiCad schematic (older format))
At the start: 20 parts, among them J1 Conn_01x05, J2 Conn_01x05, Q1 BSS138DW, Q2 BSS138DW, U1 AP2127K-3.3, U2 ADXL345

Commit message: Schematic PDF and 3D Renders added
Parts:
- removed U2: ADXL345, Package_LGA:LGA-14_3x5mm_P0.8mm_LayoutBorder1x6y, symbol ADXL345:ADXL345
- added U?: ADXL345, Package_LGA:LGA-14_3x5mm_P0.8mm_LayoutBorder1x6y, symbol SirBoard_Library:ADXL345
Changed lines of the file:
@@
 EESchema Schematic File Version 4
-LIBS:ADXL345v2-cache
 EELAYER 29 0
 EELAYER END
@@
 	6200 900  6850 900
 $Comp
-L ADXL345:ADXL345 U2
-U 1 1 5DFC1741
-P 5950 3075
-F 0 "U2" H 5937 3893 50  0000 C CNN
-F 1 "ADXL345" H 5937 3803 50  0000 C CNN
-F 2 "Package_LGA:LGA-14_3x5mm_P0.8mm_LayoutBorder1x6y" H 5950 3650 50  0001 C CNN
-F 3 "" H 5950 3650 50  0001 C CNN
-F 4 "C9667" H 5937 3713 50  0000 C CNN "Part"
-	1    5950 3075
-	1    0    0    -1
-$EndComp
-$Comp
 L Connector_Generic:Conn_01x05 J1
 U 1 1 5DF146B7
@@
 	1    0    0    -1
 $EndComp
+$Comp
+L SirBoard_Library:ADXL345 U?
+U 1 1 5E13193E
+P 5950 3075
+F 0 "U?" H 5937 3803 50  0000 C CNN
+F 1 "ADXL345" H 5937 3713 50  0000 C CNN
+F 2 "Package_LGA:LGA-14_3x5mm_P0.8mm_LayoutBorder1x6y" H 5950 3650 50  0001 C CNN
+F 3 "" H 5950 3650 50  0001 C CNN
+F 4 "C9667" H 5937 3713 50  0001 C CNN "Part"
+	1    5950 3075
+	1    0    0    -1
+$EndComp
