File: MCP4725/MCP4725.sch (KiCad schematic (older format))
At the start: 11 parts, among them J1 Conn_01x05, U1 MCP4725

Commit message: Schematic PDF and 3D Renders added
Parts:
- U1: symbol MCP4725:MCP4725 -> MCP4725-rescue:MCP4725-MCP4725
Changed lines of the file:
@@
 SDA
 $Comp
-L MCP4725:MCP4725 U1
+L MCP4725-rescue:MCP4725-MCP4725 U1
 U 1 1 5DFC84F9
 P 2975 1375
