File: MMA845X/MMA845X.sch (KiCad schematic (older format))
At the start: 18 parts, among them J1 Conn_01x04, J2 Conn_01x04, Q1 BSS138DW, U1 AP2127K-3.3, U2 MMA845X

Commit message: Part numbers added for all variants
Parts:
- U2: Part C118083 -> C118083; C11360; C122561
Changed lines of the file:
@@
 EESchema Schematic File Version 4
-LIBS:MMA8451Q-cache
+LIBS:MMA845X-cache
 EELAYER 29 0
 EELAYER END
@@
 F 2 "SirBoardLibrary:QFN-COL-16-P=0.5" H 5650 3450 50  0001 C CNN
 F 3 "" H 5650 3450 50  0001 C CNN
-F 4 "C118083" H 5650 3375 50  0001 C CNN "Part"
+F 4 "C118083; C11360; C122561" H 5650 3375 50  0001 C CNN "Part"
 	1    5650 2900
 	1    0    0    -1
